File: RFCAR/CONTROLLER/kicad/CONTROLLER.sch (KiCad schematic (older format))
At the start: 6 parts, among them U1 LM1117-3.3, U2 L7805

Commit message: kicad
Connections:
- net at U1.3 (VI), U2.3 (OUT): now also C2.1; no longer C3.1, C4.1
- net at U1.2 (VO): now also C3.1, C4.1; no longer C2.1
Other:
- moved on the sheet: C2, C3, C4, U1
Changed lines of the file:
@@
 EESchema Schematic File Version 4
+LIBS:CONTROLLER-cache
 EELAYER 26 0
 EELAYER END
@@
 L Device:CP C3
 U 1 1 5BEC95AE
-P 8050 3950
-F 0 "C3" V 8305 3950 50  0000 C CNN
-F 1 "CP" V 8214 3950 50  0000 C CNN
-F 2 "" H 8088 3800 50  0001 C CNN
-F 3 "~" H 8050 3950 50  0001 C CNN
-	1    8050 3950
+P 8650 4500
+F 0 "C3" V 8905 4500 50  0000 C CNN
+F 1 "CP" V 8814 4500 50  0000 C CNN
+F 2 "" H 8688 4350 50  0001 C CNN
+F 3 "~" H 8650 4500 50  0001 C CNN
+	1    8650 4500
 	0    -1   -1   0
 $EndComp
-Wire Wire Line
-	7750 4500 8200 4500
-Wire Wire Line
-	8200 4500 8200 3950
 $Comp
 L Regulator_Linear:LM1117-3.3 U1
 U 1 1 5BEC973C
-P 7600 3200
-F 0 "U1" H 7600 3442 50  0000 C CNN
-F 1 "LM1117-3.3" H 7600 3351 50  0000 C CNN
-F 2 "" H 7600 3200 50  0001 C CNN
-F 3 "http://www.ti.com/lit/ds/symlink/lm1117.pdf" H 7600 3200 50  0001 C CNN
-	1    7600 3200
+P 8200 3950
+F 0 "U1" H 8200 4192 50  0000 C CNN
+F 1 "LM1117-3.3" H 8200 4101 50  0000 C CNN
+F 2 "" H 8200 3950 50  0001 C CNN
+F 3 "http://www.ti.com/lit/ds/symlink/lm1117.pdf" H 8200 3950 50  0001 C CNN
+	1    8200 3950
 	1    0    0    -1
 $EndComp
@@
 L Device:CP C4
 U 1 1 5BEC976A
-P 8050 3950
-F 0 "C4" V 8305 3950 50  0000 C CNN
-F 1 "CP" V 8214 3950 50  0000 C CNN
-F 2 "" H 8088 3800 50  0001 C CNN
-F 3 "~" H 8050 3950 50  0001 C CNN
-	1    8050 3950
+P 8650 4500
+F 0 "C4" V 8905 4500 50  0000 C CNN
+F 1 "CP" V 8814 4500 50  0000 C CNN
+F 2 "" H 8688 4350 50  0001 C CNN
+F 3 "~" H 8650 4500 50  0001 C CNN
+	1    8650 4500
 	0    -1   -1   0
 $EndComp
-Connection ~ 8200 3950
-Connection ~ 7900 3950
 $Comp
 L Device:CP C2
 U 1 1 5BEC9820
-P 8050 3200
-F 0 "C2" V 8305 3200 50  0000 C CNN
-F 1 "CP" V 8214 3200 50  0000 C CNN
-F 2 "" H 8088 3050 50  0001 C CNN
-F 3 "~" H 8050 3200 50  0001 C CNN
-	1    8050 3200
+P 8050 4500
+F 0 "C2" V 8305 4500 50  0000 C CNN
+F 1 "CP" V 8214 4500 50  0000 C CNN
+F 2 "" H 8088 4350 50  0001 C CNN
+F 3 "~" H 8050 4500 50  0001 C CNN
+	1    8050 4500
 	0    -1   -1   0
 $EndComp
 Wire Wire Line
-	8200 3950 8200 3500
+	7900 3950 7900 4500
 Wire Wire Line
-	8200 3500 7600 3500
+	8200 4250 8200 4500
 Wire Wire Line
-	8200 3500 8200 3200
-Connection ~ 8200 3500
+	7750 4500 7800 4500
 Wire Wire Line
-	7900 3950 7900 3600
+	7800 4500 7800 4650
 Wire Wire Line
-	7900 3600 7300 3600
+	7800 4650 8200 4650
 Wire Wire Line
-	7300 3600 7300 3200
+	8200 4650 8200 4500
+Connection ~ 8200 4500
+Connection ~ 7900 3950
+Wire Wire Line
+	8500 3950 8500 4500
+Connection ~ 8500 4500
+Wire Wire Line
+	8200 4650 8800 4650
+Wire Wire Line
+	8800 4650 8800 4500
+Connection ~ 8200 4650
+Connection ~ 8800 4500
 $EndSCHEMATC

Commit message: kicad
Parts:
- added C5, C6: C, symbol Device:C
- added D1: LED, symbol Device:LED
- added J1: Conn_01x08_Male, symbol Connector:Conn_01x08_Male
- added J2: Conn_01x07_Male, symbol Connector:Conn_01x07_Male
- added J3: Conn_01x06_Male, symbol Connector:Conn_01x06_Male
- added J4: Conn_01x01_Male, symbol Connector:Conn_01x01_Male
- added R1: R 470, symbol Device:R
- added U3: ATmega328P-PU, Package_DIP:DIP-28_W7.62mm, symbol MCU_Microchip_ATmega:ATmega328P-PU
- added U4: ADG417BN, Package_DIP:DIP-8_W7.62mm, symbol Analog_Switch:ADG417BN
- added Y1: Crystal, symbol Device:Crystal
Connections:
- net +9V: now also U4.1
- net GND: now also C5.1, C6.1, D1.1 (K), U3.22 (GND), U3.8 (GND), U4.6, U4.8
- net at C2.1, U1.3 (VI), U2.3 (OUT): now also R1.2, U3.20 (AVCC), U3.7 (VCC)
- new net: J2.1 (Pin_1), U3.1 (~RESET~/PC6)
- new net: C5.2, U3.10 (XTAL2/PB7), Y1.1
- new net: J1.3 (Pin_3), U3.11 (PD5)
- new net: J1.2 (Pin_2), U3.12 (PD6)
- new net: J1.1 (Pin_1), U3.13 (PD7)
- new net: J3.6 (Pin_6), U3.14 (PB0)
- new net: J3.5 (Pin_5), U3.15 (PB1)
- new net: J3.4 (Pin_4), U3.16 (PB2)
- new net: J3.3 (Pin_3), U3.17 (PB3)
- new net: J3.2 (Pin_2), U3.18 (PB4)
- new net: J3.1 (Pin_1), U3.19 (PB5)
- new net: J1.8 (Pin_8), U3.2 (PD0)
- new net: J4.1 (Pin_1), U3.21 (AREF)
- new net: J2.7 (Pin_7), U3.23 (PC0)
- new net: J2.6 (Pin_6), U3.24 (PC1)
- new net: J2.5 (Pin_5), U3.25 (PC2)
- new net: J2.4 (Pin_4), U3.26 (PC3)
- new net: J2.3 (Pin_3), U3.27 (PC4)
- new net: J2.2 (Pin_2), U3.28 (PC5)
- new net: J1.7 (Pin_7), U3.3 (PD1)
- new net: J1.6 (Pin_6), U3.4 (PD2)
- new net: J1.5 (Pin_5), U3.5 (PD3)
- new net: J1.4 (Pin_4), U3.6 (PD4)
- new net: C6.2, U3.9 (XTAL1/PB6), Y1.2
- new net: D1.2 (A), R1.1
Changed lines of the file:
@@
 L power:+9V #PWR0103
 U 1 1 5BEC938E
-P 7450 4700
-F 0 "#PWR0103" H 7450 4550 50  0001 C CNN
-F 1 "+9V" H 7465 4873 50  0000 C CNN
-F 2 "" H 7450 4700 50  0001 C CNN
-F 3 "" H 7450 4700 50  0001 C CNN
-	1    7450 4700
+P 7300 5250
+F 0 "#PWR0103" H 7300 5100 50  0001 C CNN
+F 1 "+9V" H 7315 5423 50  0000 C CNN
+F 2 "" H 7300 5250 50  0001 C CNN
+F 3 "" H 7300 5250 50  0001 C CNN
+	1    7300 5250
 	-1   0    0    1
 $EndComp
@@
 L power:GND #PWR0104
 U 1 1 5BEC93B7
-P 7750 4700
-F 0 "#PWR0104" H 7750 4450 50  0001 C CNN
-F 1 "GND" H 7755 4527 50  0000 C CNN
-F 2 "" H 7750 4700 50  0001 C CNN
-F 3 "" H 7750 4700 50  0001 C CNN
-	1    7750 4700
+P 7600 5450
+F 0 "#PWR0104" H 7600 5200 50  0001 C CNN
+F 1 "GND" H 7605 5277 50  0000 C CNN
+F 2 "" H 7600 5450 50  0001 C CNN
+F 3 "" H 7600 5450 50  0001 C CNN
+	1    7600 5450
 	1    0    0    -1
 $EndComp
@@
 Connection ~ 8200 4650
 Connection ~ 8800 4500
+$Comp
+L Device:Crystal Y1
+U 1 1 5BF5DD23
+P 8350 3400
+F 0 "Y1" H 8350 3668 50  0000 C CNN
+F 1 "Crystal" H 8350 3577 50  0000 C CNN
+F 2 "" H 8350 3400 50  0001 C CNN
+F 3 "~" H 8350 3400 50  0001 C CNN
+	1    8350 3400
+	1    0    0    -1
+$EndComp
+Wire Wire Line
+	8200 3400 8200 3200
+Wire Wire Line
+	8200 3200 8350 3200
+Wire Wire Line
+	8450 3200 8500 3200
+Wire Wire Line
+	8500 3200 8500 3400
+$Comp
+L Device:C C5
+U 1 1 5BF5E25F
+P 9050 4500
+F 0 "C5" V 8798 4500 50  0000 C CNN
+F 1 "C" V 8889 4500 50  0000 C CNN
+F 2 "" H 9088 4350 50  0001 C CNN
+F 3 "~" H 9050 4500 50  0001 C CNN
+	1    9050 4500
+	0    1    1    0
+$EndComp
+Wire Wire Line
+	8800 4650 9200 4650
+Wire Wire Line
+	9200 4650 9200 4500
+Connection ~ 8800 4650
+$Comp
+L Device:C C6
+U 1 1 5BF5E6DE
+P 9450 4500
+F 0 "C6" V 9198 4500 50  0000 C CNN
+F 1 "C" V 9289 4500 50  0000 C CNN
+F 2 "" H 9488 4350 50  0001 C CNN
+F 3 "~" H 9450 4500 50  0001 C CNN
+	1    9450 4500
+	0    1    1    0
+$EndComp
+Wire Wire Line
+	9200 4650 9600 4650
+Wire Wire Line
+	9600 4650 9600 4500
+Connection ~ 9200 4650
+Wire Wire Line
+	8200 3400 8200 3600
+Wire Wire Line
+	8200 3600 8900 3600
+Wire Wire Line
+	8900 3600 8900 4500
+Connection ~ 8200 3400
+Wire Wire Line
+	8500 3400 9300 3400
+Wire Wire Line
+	9300 3400 9300 4500
+Connection ~ 8500 3400
+Wire Wire Line
+	8350 2600 8350 3200
+$Comp
+L MCU_Microchip_ATmega:ATmega328P-PU U3
+U 1 1 5BF46BC3
+P 7850 2000
+F 0 "U3" V 7072 2000 50  0000 C CNN
+F 1 "ATmega328P-PU" V 7163 2000 50  0000 C CNN
+F 2 "Package_DIP:DIP-28_W7.62mm" H 7850 2000 50  0001 C CIN
+F 3 "http://ww1.microchip.com/downloads/en/DeviceDoc/ATmega328_P%20AVR%20MCU%20with%20picoPower%20Technology%20Data%20Sheet%2040001984A.pdf" H 7850 2000 50  0001 C CNN
+	1    7850 2000
+	0    1    1    0
+$EndComp
+Wire Wire Line
+	9600 4500 9600 600
+Wire Wire Line
+	9600 600  9050 600
+Wire Wire Line
+	6100 600  6100 2000
+Wire Wire Line
+	6100 2000 6350 2000
+Connection ~ 9600 4500
+Wire Wire Line
+	7900 3950 7900 3000
+$Comp
+L Connector:Conn_01x01_Male J4
+U 1 1 5BF63996
+P 9050 1200
+F 0 "J4" V 9110 1240 50  0000 L CNN
+F 1 "Conn_01x01_Male" V 9201 1240 50  0000 L CNN
+F 2 "" H 9050 1200 50  0001 C CNN
+F 3 "~" H 9050 1200 50  0001 C CNN
+	1    9050 1200
+	0    1    1    0
+$EndComp
+$Comp
+L Connector:Conn_01x06_Male J3
+U 1 1 5BF64068
+P 8750 2800
+F 0 "J3" V 8903 2413 50  0000 R CNN
+F 1 "Conn_01x06_Male" V 8812 2413 50  0000 R CNN
+F 2 "" H 8750 2800 50  0001 C CNN
+F 3 "~" H 8750 2800 50  0001 C CNN
+	1    8750 2800
+	0    -1   -1   0
+$EndComp
+$Comp
+L Connector:Conn_01x07_Male J2
+U 1 1 5BF64106
+P 7850 2800
+F 0 "J2" V 7778 2777 50  0000 C CNN
+F 1 "Conn_01x07_Male" V 7687 2777 50  0000 C CNN
+F 2 "" H 7850 2800 50  0001 C CNN
+F 3 "~" H 7850 2800 50  0001 C CNN
+	1    7850 2800
+	0    -1   -1   0
+$EndComp
+Wire Wire Line
+	7900 3000 9350 3000
+$Comp
+L Connector:Conn_01x08_Male J1
+U 1 1 5BF658B0
+P 6950 2800
+F 0 "J1" V 6878 2727 50  0000 C CNN
+F 1 "Conn_01x08_Male" V 6787 2727 50  0000 C CNN
+F 2 "" H 6950 2800 50  0001 C CNN
+F 3 "~" H 6950 2800 50  0001 C CNN
+	1    6950 2800
+	0    -1   -1   0
+$EndComp
+Wire Wire Line
+	8450 3200 8450 2600
+Wire Wire Line
+	9350 3000 9350 2100
+Connection ~ 9350 2100
+$Comp
+L Device:LED D1
+U 1 1 5BF6873C
+P 9200 800
+F 0 "D1" H 9191 1016 50  0000 C CNN
+F 1 "LED" H 9191 925 50  0000 C CNN
+F 2 "" H 9200 800 50  0001 C CNN
+F 3 "~" H 9200 800 50  0001 C CNN
+	1    9200 800
+	1    0    0    -1
+$EndComp
+Wire Wire Line
+	9050 800  9050 600
+Connection ~ 9050 600
+Wire Wire Line
+	9050 600  6100 600
+Wire Wire Line
+	9350 2000 9350 2100
+$Comp
+L Device:R R1
+U 1 1 5BF6BD52
+P 9350 950
+F 0 "R1" H 9420 996 50  0000 L CNN
+F 1 "R 470" H 9420 905 50  0000 L CNN
+F 2 "" V 9280 950 50  0001 C CNN
+F 3 "~" H 9350 950 50  0001 C CNN
+	1    9350 950
+	1    0    0    -1
+$EndComp
+Wire Wire Line
+	9350 1100 9350 2000
+Connection ~ 9350 2000
+$Comp
+L Analog_Switch:ADG417BN U4
+U 1 1 5BF6D5EA
+P 7600 5250
+F 0 "U4" H 7600 5517 50  0000 C CNN
+F 1 "ADG417BN" H 7600 5426 50  0000 C CNN
+F 2 "Package_DIP:DIP-8_W7.62mm" H 7600 5150 50  0001 C CNN
+F 3 "http://www.analog.com/media/en/technical-documentation/data-sheets/ADG417.pdf" H 7600 5250 50  0001 C CNN
+	1    7600 5250
+	1    0    0    -1
+$EndComp
+Wire Wire Line
+	7600 5450 7900 5450
+Wire Wire Line
+	7900 5450 7900 5250
+Connection ~ 7600 5450
+Wire Wire Line
+	7900 5250 7900 4700
+Wire Wire Line
+	7900 4700 7750 4700
+Connection ~ 7900 5250
+Wire Wire Line
+	7450 4700 7300 4700
+Wire Wire Line
+	7300 4700 7300 5250
+Connection ~ 7300 5250
 $EndSCHEMATC

Commit message: kicad
Parts:
- removed C4: CP, symbol Device:CP
- removed C6: C, symbol Device:C
- removed J1: Conn_01x08_Male, symbol Connector:Conn_01x08_Male
- removed J2: Conn_01x07_Male, symbol Connector:Conn_01x07_Male
- removed J3: Conn_01x06_Male, symbol Connector:Conn_01x06_Male
- removed J4: Conn_01x01_Male, symbol Connector:Conn_01x01_Male
- removed U1: LM1117-3.3, symbol Regulator_Linear:LM1117-3.3
- removed U2: L7805, symbol Regulator_Linear:L7805
- removed U3: ATmega328P-PU, Package_DIP:DIP-28_W7.62mm, symbol MCU_Microchip_ATmega:ATmega328P-PU
- removed U4: ADG417BN, Package_DIP:DIP-8_W7.62mm, symbol Analog_Switch:ADG417BN
- added BT1: Battery_Cell, symbol Device:Battery_Cell
- added C4: C, Capacitor_THT:C_Axial_L3.8mm_D2.6mm_P7.50mm_Horizontal, symbol Device:C
- added JT01_5V1, JT01_BT1, JT01_GND1, JT01_X1, JT01_Y1, JT02_5V1, JT02_BT1, JT02_GND1, JT02_X1, JT02_Y1, _1, _10, _11, _2, _3, _4, _5, _6, _7, _8, _9, nrf_CE_PB1_09D1, nrf_CSN_PB2_10D1, nrf_GND1, nrf_MISO_PB4_12D1, nrf_MOSI_PB3_11D1, nrf_SCK_PB5_13D1, nrf_V+_3.3: (no value), Connector_PinHeader_2.00mm:PinHeader_1x01_P2.00mm_Vertical, symbol Connector:Conn_01x01_Female
- added U1: LM7805_TO220, Converter_DCDC:Converter_DCDC_TRACO_TSR-1_THT, symbol Regulator_Linear:LM7805_TO220
- added U2: ATmega328-PU, Package_DIP:DIP-28_W7.62mm, symbol MCU_Microchip_ATmega:ATmega328-PU
- added U3: LM1117-3.3, Converter_DCDC:Converter_DCDC_TRACO_TSR-1_THT, symbol Regulator_Linear:LM1117-3.3
- C1, C2, C3, C5: footprint (none) -> Capacitor_THT:C_Axial_L3.8mm_D2.6mm_P7.50mm_Horizontal
- R1: value R 470 -> R
- Y1: footprint (none) -> Crystal:Crystal_HC49-U_Vertical
Connections:
- net +9V: now also BT1.1 (+), U1.1 (VI)
- net GND: now also R1.2, BT1.2 (-), C4.1, JT01_GND1.1 (Pin_1), JT02_GND1.1 (Pin_1), U1.2 (GND), U2.22 (GND), U2.8 (GND), U3.1 (GND), nrf_GND1.1 (Pin_1); no longer D1.1 (K)
- net at C2.1: now also D1.1 (K), JT01_5V1.1 (Pin_1), JT02_5V1.1 (Pin_1), U1.3 (VO), U2.20 (AVCC), U2.7 (VCC), U3.3 (VI); no longer R1.2
- net at C3.1: now also U3.2 (VO), nrf_V+_3.3.1 (Pin_1)
- net at C5.2: now also Y1.2, U2.10 (XTAL2/PB7); no longer Y1.1
- new net: U2.1 (~RESET~/PC6), _4.1 (Pin_1)
- new net: U2.11 (PD5), _8.1 (Pin_1)
- new net: U2.12 (PD6), _9.1 (Pin_1)
- new net: U2.13 (PD7), _10.1 (Pin_1)
- new net: U2.14 (PB0), _1.1 (Pin_1)
- new net: U2.15 (PB1), nrf_CE_PB1_09D1.1 (Pin_1)
- new net: U2.16 (PB2), nrf_CSN_PB2_10D1.1 (Pin_1)
- new net: U2.17 (PB3), nrf_MOSI_PB3_11D1.1 (Pin_1)
- new net: U2.18 (PB4), nrf_MISO_PB4_12D1.1 (Pin_1)
- new net: U2.19 (PB5), nrf_SCK_PB5_13D1.1 (Pin_1)
- new net: U2.2 (PD0), _5.1 (Pin_1)
- new net: U2.21 (AREF), _11.1 (Pin_1)
- new net: JT01_X1.1 (Pin_1), U2.23 (PC0)
- new net: JT01_Y1.1 (Pin_1), U2.24 (PC1)
- new net: JT02_X1.1 (Pin_1), U2.25 (PC2)
- new net: JT02_Y1.1 (Pin_1), U2.26 (PC3)
- new net: U2.27 (PC4), _2.1 (Pin_1)
- new net: U2.28 (PC5), _3.1 (Pin_1)
- new net: U2.3 (PD1), _6.1 (Pin_1)
- new net: JT01_BT1.1 (Pin_1), U2.4 (PD2)
- new net: JT02_BT1.1 (Pin_1), U2.5 (PD3)
- new net: U2.6 (PD4), _7.1 (Pin_1)
- new net: C4.2, U2.9 (XTAL1/PB6), Y1.1
