File: RFCAR/CONTROLLER/kicad/CONTROLLER/CONTROLLER.sch (KiCad schematic (older format))
At the start: 41 parts, among them J1 XLR3_Switched, U1 LM7805_TO220, U2 ATmega328-PU, U3 LM1117-3.3, Y1 Crystal

Commit message: hardware
Parts:
- removed J1: XLR3_Switched, symbol Connector:XLR3_Switched
- added SW1: SW_DIP_x01, symbol switch:SW_DIP_x01
Connections:
- net labels added: +3.3V, +5V, +BATT
- wire segments 48 -> 49
Other:
- moved on the sheet: BT1
Changed lines of the file:
@@
 EESchema Schematic File Version 4
+LIBS:CONTROLLER-cache
 EELAYER 26 0
 EELAYER END
@@
 $EndComp
 $Comp
-L power:+9V #PWR06
-U 1 1 5BFBE081
-P 5300 650
-F 0 "#PWR06" H 5300 500 50  0001 C CNN
-F 1 "+9V" H 5315 823 50  0000 C CNN
-F 2 "" H 5300 650 50  0001 C CNN
-F 3 "" H 5300 650 50  0001 C CNN
-	1    5300 650
-	1    0    0    -1
-$EndComp
-$Comp
 L Device:CP C1
 U 1 1 5BFBE174
@@
 L Device:Battery_Cell BT1
 U 1 1 5BFDC488
-P 5200 1750
-F 0 "BT1" V 4945 1800 50  0000 C CNN
-F 1 "Battery_Cell" V 5036 1800 50  0000 C CNN
-F 2 "" V 5200 1810 50  0001 C CNN
-F 3 "~" V 5200 1810 50  0001 C CNN
-	1    5200 1750
+P 5200 950
+F 0 "BT1" V 4945 1000 50  0000 C CNN
+F 1 "Battery_Cell" V 5036 1000 50  0000 C CNN
+F 2 "" V 5200 1010 50  0001 C CNN
+F 3 "~" V 5200 1010 50  0001 C CNN
+	1    5200 950
 	0    1    1    0
 $EndComp
@@
 L power:GND #PWR03
 U 1 1 5BFE27A5
-P 5100 1750
-F 0 "#PWR03" H 5100 1500 50  0001 C CNN
-F 1 "GND" H 5105 1577 50  0000 C CNN
-F 2 "" H 5100 1750 50  0001 C CNN
-F 3 "" H 5100 1750 50  0001 C CNN
-	1    5100 1750
+P 5100 950
+F 0 "#PWR03" H 5100 700 50  0001 C CNN
+F 1 "GND" H 5105 777 50  0000 C CNN
+F 2 "" H 5100 950 50  0001 C CNN
+F 3 "" H 5100 950 50  0001 C CNN
+	1    5100 950
 	1    0    0    -1
 $EndComp
@@
 Wire Wire Line
 	7050 2250 7050 2550
-$Comp
-L power:GND #PWR07
-U 1 1 5C0615FA
-P 5200 1250
-F 0 "#PWR07" H 5200 1000 50  0001 C CNN
-F 1 "GND" H 5205 1077 50  0000 C CNN
-F 2 "" H 5200 1250 50  0001 C CNN
-F 3 "" H 5200 1250 50  0001 C CNN
-	1    5200 1250
-	1    0    0    -1
-$EndComp
-$Comp
-L Connector:XLR3_Switched J1
-U 2 1 5C062CDA
-P 5300 950
-F 0 "J1" V 5254 1154 50  0000 L CNN
-F 1 "XLR3_Switched" V 5345 1154 50  0000 L CNN
-F 2 "" H 5300 1050 50  0001 C CNN
-F 3 " ~" H 5300 1050 50  0001 C CNN
-	2    5300 950
-	0    1    1    0
-$EndComp
+Wire Wire Line
+	5400 950  5400 1350
+Wire Wire Line
+	5400 2250 5400 2400
+$Comp
+L power:+BATT #PWR0101
+U 1 1 5C06009C
+P 1550 7550
+F 0 "#PWR0101" H 1550 7400 50  0001 C CNN
+F 1 "+BATT" H 1565 7723 50  0000 C CNN
+F 2 "" H 1550 7550 50  0001 C CNN
+F 3 "" H 1550 7550 50  0001 C CNN
+	1    1550 7550
+	-1   0    0    1
+$EndComp
+$Comp
+L power:PWR_FLAG #FLG0101
+U 1 1 5C063F8F
+P 1550 7550
+F 0 "#FLG0101" H 1550 7625 50  0001 C CNN
+F 1 "PWR_FLAG" H 1550 7724 50  0000 C CNN
+F 2 "" H 1550 7550 50  0001 C CNN
+F 3 "~" H 1550 7550 50  0001 C CNN
+	1    1550 7550
+	1    0    0    -1
+$EndComp
+$Comp
+L power:PWR_FLAG #FLG0102
+U 1 1 5C0667BA
+P 2000 7550
+F 0 "#FLG0102" H 2000 7625 50  0001 C CNN
+F 1 "PWR_FLAG" H 2000 7724 50  0000 C CNN
+F 2 "" H 2000 7550 50  0001 C CNN
+F 3 "~" H 2000 7550 50  0001 C CNN
+	1    2000 7550
+	1    0    0    -1
+$EndComp
+$Comp
+L power:+5V #PWR0102
+U 1 1 5C0674CE
+P 2000 7550
+F 0 "#PWR0102" H 2000 7400 50  0001 C CNN
+F 1 "+5V" H 2015 7723 50  0000 C CNN
+F 2 "" H 2000 7550 50  0001 C CNN
+F 3 "" H 2000 7550 50  0001 C CNN
+	1    2000 7550
+	-1   0    0    1
+$EndComp
+$Comp
+L power:PWR_FLAG #FLG0103
+U 1 1 5C067584
+P 2450 7550
+F 0 "#FLG0103" H 2450 7625 50  0001 C CNN
+F 1 "PWR_FLAG" H 2450 7724 50  0000 C CNN
+F 2 "" H 2450 7550 50  0001 C CNN
+F 3 "~" H 2450 7550 50  0001 C CNN
+	1    2450 7550
+	1    0    0    -1
+$EndComp
+$Comp
+L power:+3.3V #PWR0103
+U 1 1 5C067682
+P 2450 7550
+F 0 "#PWR0103" H 2450 7400 50  0001 C CNN
+F 1 "+3.3V" H 2465 7723 50  0000 C CNN
+F 2 "" H 2450 7550 50  0001 C CNN
+F 3 "" H 2450 7550 50  0001 C CNN
+	1    2450 7550
+	-1   0    0    1
+$EndComp
+Wire Wire Line
+	5400 2250 5400 1950
 Connection ~ 5400 2250
-Wire Wire Line
-	5400 2250 5400 2400
-Connection ~ 5400 1750
-Wire Wire Line
-	5400 1750 5400 2250
-Wire Wire Line
-	5400 1250 5400 1750
+$Comp
+L power:+9V #PWR0104
+U 1 1 5C05DB23
+P 5400 700
+F 0 "#PWR0104" H 5400 550 50  0001 C CNN
+F 1 "+9V" H 5415 873 50  0000 C CNN
+F 2 "" H 5400 700 50  0001 C CNN
+F 3 "" H 5400 700 50  0001 C CNN
+	1    5400 700
+	1    0    0    -1
+$EndComp
+Wire Wire Line
+	5400 950  5400 700
+Connection ~ 5400 950
+$Comp
+L switch:SW_DIP_x01 SW1
+U 1 1 5C081EE9
+P 5400 1650
+F 0 "SW1" V 5354 1780 50  0000 L CNN
+F 1 "SW_DIP_x01" V 5445 1780 50  0000 L CNN
+F 2 "" H 5400 1650 50  0001 C CNN
+F 3 "" H 5400 1650 50  0001 C CNN
+	1    5400 1650
+	0    1    1    0
+$EndComp
 $EndSCHEMATC
